Commit message: added custom base to elevate robot

File: src/kuka_barrett_description/urdf/iiwa.gazebo.xacro (robot description, xacro)
@@ -8,4 +8,10 @@
       </plugin>
     </gazebo-->
+    <!-- robot_base -->
+    <gazebo reference="custom_base">
+      <material>Gazebo/Grey</material>
+      <mu1>0.2</mu1>
+      <mu2>0.2</mu2>
+    </gazebo>
     <!-- Link0 -->
     <gazebo reference="${robot_name}_link_0">

File: src/kuka_barrett_description/urdf/iiwa14.xacro (robot description, xacro)
@@ -14,8 +14,37 @@
   <xacro:property name="max_velocity" value="10"/>
   <xacro:macro name="iiwa14" params="parent hardware_interface robot_name *origin">
-    <!--joint between {parent} and link_0-->
-    <joint name="${parent}_${robot_name}_joint" type="fixed">
+    <!--joint between {parent} (world) and custom_base-->
+    <joint name="${parent}_custom_base_joint" type="fixed">
       <xacro:insert_block name="origin"/>
       <parent link="${parent}"/>
+      <child link="custom_base"/>
+    </joint>
+    <!-- Robot base -->
+    <link name="custom_base">
+      <inertial>
+        <origin xyz="0 0 0" rpy="0 0 0"/>
+        <mass value="10"/>
+        <inertia ixx="100"  ixy="0"  ixz="0" iyy="100" iyz="0" izz="100" />
+      </inertial>
+      <visual>
+        <origin xyz="0 0 0.4110095" rpy="0 0 0" />
+        <geometry>
+          <box size="0.483711 0.509896 0.822019" />
+        </geometry>
+        <material name="Cyan">
+          <color rgba="0 1.0 1.0 1.0"/>
+        </material>
+      </visual>
+      <collision>
+        <origin xyz="0 0 0.4110095" rpy="0 0 0"/>
+        <geometry>
+          <box size="0.483711 0.509896 0.822019" />
+        </geometry>
+      </collision>
+    </link>
+    <!--joint between base and link_0-->
+    <joint name="custom_base_${robot_name}_joint" type="fixed">
+      <origin xyz="0 0 0.822019" rpy="0 0 0"/>
+      <parent link="custom_base"/>
       <child link="${robot_name}_link_0"/>
     </joint>

File: src/kuka_barrett_description/urdf/kuka_barrett.xacro.urdf (robot description, URDF)
Before this commit: robot kuka_barrett, 20 links, 19 joints
Links:
- added link custom_base, mass 10; collision box size=0.483711 0.509896 0.822019; visual box size=0.483711 0.509896 0.822019
- link bh_base_link: geometry collision mesh filename=package://kuka_barrett_description/meshes/palm_282.dae; visual mesh filename=package://kuka_barrett_description/meshes/palm_282.dae
- link bh_finger_11_link: geometry collision mesh filename=package://kuka_barrett_description/meshes/knuckle.dae; visual mesh filename=package://kuka_barrett_description/meshes/knuckle.dae
- link bh_finger_12_link: geometry collision mesh filename=package://kuka_barrett_description/meshes/finger.dae; visual mesh filename=package://kuka_barrett_description/meshes/finger.dae
- link bh_finger_13_link: geometry collision mesh filename=package://kuka_barrett_description/meshes/finger_tip.dae; visual mesh filename=package://kuka_barrett_description/meshes/finger_tip.dae
- link bh_finger_21_link: geometry collision mesh filename=package://kuka_barrett_description/meshes/knuckle.dae; visual mesh filename=package://kuka_barrett_description/meshes/knuckle.dae
- link bh_finger_22_link: geometry collision mesh filename=package://kuka_barrett_description/meshes/finger.dae; visual mesh filename=package://kuka_barrett_description/meshes/finger.dae
- link bh_finger_23_link: geometry collision mesh filename=package://kuka_barrett_description/meshes/finger_tip.dae; visual mesh filename=package://kuka_barrett_description/meshes/finger_tip.dae
- link bh_finger_31_link: geometry collision mesh filename=package://kuka_barrett_description/meshes/knuckle_fixed.dae; visual mesh filename=package://kuka_barrett_description/meshes/knuckle_fixed.dae
- link bh_finger_32_link: geometry collision mesh filename=package://kuka_barrett_description/meshes/finger.dae; visual mesh filename=package://kuka_barrett_description/meshes/finger.dae
- link bh_finger_33_link: geometry collision mesh filename=package://kuka_barrett_description/meshes/finger_tip.dae; visual mesh filename=package://kuka_barrett_description/meshes/finger_tip.dae
- link iiwa_link_0: geometry collision mesh filename=package://kuka_barrett_description/meshes/iiwa14/collision/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; visual mesh filename=package://kuka_barrett_description/meshes/iiwa14/visual/lin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
- link iiwa_link_1: geometry collision mesh filename=package://kuka_barrett_description/meshes/iiwa14/collision/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; visual mesh filename=package://kuka_barrett_description/meshes/iiwa14/visual/lin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
- link iiwa_link_2: geometry collision mesh filename=package://kuka_barrett_description/meshes/iiwa14/collision/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; visual mesh filename=package://kuka_barrett_description/meshes/iiwa14/visual/lin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
- link iiwa_link_3: geometry collision mesh filename=package://kuka_barrett_description/meshes/iiwa14/collision/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; visual mesh filename=package://kuka_barrett_description/meshes/iiwa14/visual/lin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
- link iiwa_link_4: geometry collision mesh filename=package://kuka_barrett_description/meshes/iiwa14/collision/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; visual mesh filename=package://kuka_barrett_description/meshes/iiwa14/visual/lin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
- link iiwa_link_5: geometry collision mesh filename=package://kuka_barrett_description/meshes/iiwa14/collision/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; visual mesh filename=package://kuka_barrett_description/meshes/iiwa14/visual/lin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
- link iiwa_link_6: geometry collision mesh filename=package://kuka_barrett_description/meshes/iiwa14/collision/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; visual mesh filename=package://kuka_barrett_description/meshes/iiwa14/visual/lin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
- link iiwa_link_7: geometry collision mesh filename=package://kuka_barrett_description/meshes/iiwa14/collision/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; visual mesh filename=package://kuka_barrett_description/meshes/iiwa14/visual/lin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
Joints:
- removed joint world_iiwa_joint
- added joint custom_base_iiwa_joint: type fixed, parent custom_base, child iiwa_link_0, origin xyz=0 0 0.822019 rpy=0 0 0
- added joint world_custom_base_joint: type fixed, parent world, child custom_base, origin xyz=0 0 0 rpy=0 0 0
