Commit message: added camera object

File: src/kuka_barrett_description/urdf/kuka_barrett.xacro.urdf (robot description, URDF)
Before this commit: robot kuka_barrett, 21 links, 20 joints
Links:
- added link camera_link, mass 1e-5; collision box size=0.05 0.05 0.05; visual box size=0.05 0.05 0.05
Joints:
- added joint camera_joint: type fixed, parent iiwa_link_ee, child camera_link, origin xyz=0.05 0 0 rpy=0 0 0, axis 0 1 0
