Commit message: configure camera pose

File: src/kuka_barrett_description/urdf/hand_camera.xacro (robot description, xacro)
@@ -4,5 +4,5 @@
     <joint name="camera_joint" type="fixed">
         <axis xyz="0 1 0" />
-        <origin xyz="${camera_link} 0 0" rpy="0 0 0"/>
+        <origin xyz="0 0 ${2*camera_link}" rpy="0 -1.57 0"/>
         <parent link="${parent}"/>
         <child link="camera_link"/>
@@ -12,5 +12,5 @@
 				<origin xyz="0 0 0" rpy="0 0 0"/>
 				<geometry>
-					<box size="${camera_link} ${camera_link} ${camera_link}"/>
+					<box size="${camera_link/2} ${camera_link} ${camera_link}"/>
 				</geometry>
 			</collision>
@@ -18,5 +18,5 @@
 				<origin xyz="0 0 0" rpy="0 0 0"/>
 				<geometry>
-					<box size="${camera_link} ${camera_link} ${camera_link}"/>
+					<box size="${camera_link/2} ${camera_link} ${camera_link}"/>
 				</geometry>
 				<material name="red"/>

File: src/kuka_barrett_description/urdf/kuka_barrett.xacro.urdf (robot description, URDF)
Before this commit: robot kuka_barrett, 22 links, 21 joints
Links:
- link camera_link: geometry collision box size=0.025 0.05 0.05; visual box size=0.025 0.05 0.05
Joints:
- joint camera_joint: origin xyz=0.05 0 0 rpy=0 0 0 -> xyz=0 0 0.1 rpy=0.785 0 0

Commit message: small world and moveit changes

File: src/kuka_barrett_description/urdf/hand_camera.xacro (robot description, xacro)
@@ -4,5 +4,5 @@
     <joint name="camera_joint" type="fixed">
         <axis xyz="0 1 0" />
-        <origin xyz="0 0 ${2*camera_link}" rpy="0 -1.57 0"/>
+        <origin xyz="0 0 ${camera_link}" rpy="0 -1.57 0"/>
         <parent link="${parent}"/>
         <child link="camera_link"/>

File: src/kuka_barrett_description/urdf/iiwa14.xacro (robot description, xacro)
@@ -324,5 +324,5 @@
       <parent link="${robot_name}_link_7"/>
       <child link="${robot_name}_link_ee"/>
-      <origin xyz="0 0 0.045" rpy="0 0 0"/>
+      <origin xyz="0 0 0" rpy="0 0 0"/>
     </joint>
     <link name="${robot_name}_link_ee">

Commit message: Attach surgical tool to robot instead of grasping (temporary solution)

File: src/kuka_barrett_description/urdf/hand_camera.xacro (robot description, xacro)
@@ -4,7 +4,8 @@
     <joint name="camera_joint" type="fixed">
         <axis xyz="0 1 0" />
-        <origin xyz="0 0 ${camera_link}" rpy="0 -1.57 0"/>
+        <origin xyz="-${2*camera_link} 0 0" rpy="0 -1.57 0"/>
         <parent link="${parent}"/>
         <child link="camera_link"/>
+				<mimic joint="bh_base_joint" multiplier="1" offset="0"/>
     </joint>
     <link name="camera_link">

File: src/kuka_barrett_description/urdf/kuka_barrett.xacro (robot description, xacro)
@@ -14,4 +14,7 @@
   <xacro:hand_camera parent="iiwa_link_ee" camera_link="0.05" />
   <xacro:hand_camera_gazebo/>
+  <!-- Attach surgical tool for testing purposes (Instead of picking it with gripper) -->
+  <xacro:include filename="$(find kuka_barrett_description)/urdf/surgical_tool.xacro"/>
+  <xacro:surgical_tool parent="bh_base_link" />
   <gazebo>
     <plugin name="gazebo_ros_control" filename="libgazebo_ros_control.so">

Commit message: added second camera

File: src/kuka_barrett_description/urdf/hand_camera.xacro (robot description, xacro)
@@ -1,17 +1,18 @@
 <?xml version="1.0"?>
 <robot xmlns:xacro="http://www.ros.org/wiki/xacro">
-  <xacro:macro name="hand_camera" params="parent camera_link">
-    <joint name="camera_joint" type="fixed">
+  <xacro:macro name="hand_camera" params="parent camera_size">
+		<!-- Left camera -->
+    <joint name="camera_joint1" type="fixed">
         <axis xyz="0 1 0" />
-        <origin xyz="-${2*camera_link} 0 0" rpy="0 -1.57 0"/>
+        <origin xyz="-${2*camera_size} -${camera_size/2} 0" rpy="0 -1.57 0"/>
         <parent link="${parent}"/>
-        <child link="camera_link"/>
+        <child link="camera_link1"/>
 				<mimic joint="bh_base_joint" multiplier="1" offset="0"/>
     </joint>
-    <link name="camera_link">
+    <link name="camera_link1">
 			<collision>
 				<origin xyz="0 0 0" rpy="0 0 0"/>
 				<geometry>
-					<box size="${camera_link/2} ${camera_link} ${camera_link}"/>
+					<box size="${camera_size/2} ${camera_size} ${camera_size}"/>
 				</geometry>
 			</collision>
@@ -19,5 +20,5 @@
 				<origin xyz="0 0 0" rpy="0 0 0"/>
 				<geometry>
-					<box size="${camera_link/2} ${camera_link} ${camera_link}"/>
+					<box size="${camera_size/2} ${camera_size} ${camera_size}"/>
 				</geometry>
 				<material name="red"/>
@@ -30,4 +31,33 @@
 			<kinematic>1</kinematic>
     </link>
+		<!-- Right camera -->
+    <joint name="camera_joint2" type="fixed">
+        <axis xyz="0 1 0" />
+        <origin xyz="-${2*camera_size} ${camera_size/2} 0" rpy="0 -1.57 0"/>
+        <parent link="${parent}"/>
+        <child link="camera_link2"/>
+				<mimic joint="bh_base_joint" multiplier="1" offset="0"/>
+    </joint>
+    <link name="camera_link2">
+			<collision>
+				<origin xyz="0 0 0" rpy="0 0 0"/>
+				<geometry>
+					<box size="${camera_size/2} ${camera_size} ${camera_size}"/>
+				</geometry>
+			</collision>
+			<visual>
+				<origin xyz="0 0 0" rpy="0 0 0"/>
+				<geometry>
+					<box size="${camera_size/2} ${camera_size} ${camera_size}"/>
+				</geometry>
+				<material name="blue"/>
+			</visual>
+			<inertial>
+				<mass value="1e-5" />
+				<origin xyz="0 0 0" rpy="0 0 0"/>
+				<inertia ixx="1e-6" ixy="0" ixz="0" iyy="1e-6" iyz="0" izz="1e-6" />
+			</inertial>
+			<kinematic>1</kinematic>
+    </link>
   </xacro:macro>
 </robot>

File: src/kuka_barrett_description/urdf/kuka_barrett.xacro (robot description, xacro)
@@ -13,5 +13,5 @@
   <xacro:include filename="$(find kuka_barrett_description)/urdf/hand_camera.xacro"/>
   <xacro:include filename="$(find kuka_barrett_description)/urdf/hand_camera.gazebo"/>
-  <xacro:hand_camera parent="iiwa_link_ee" camera_link="0.05" />
+  <xacro:hand_camera parent="iiwa_link_ee" camera_size="0.04" />
   <xacro:hand_camera_gazebo/>
   <!-- Attach surgical tool for testing purposes (Instead of picking it with gripper)

File: src/kuka_barrett_description/urdf/kuka_barrett.xacro.urdf (robot description, URDF)
Before this commit: robot kuka_barrett, 22 links, 21 joints
Links:
- removed link camera_link
- added link camera_link1, mass 1e-5; collision box size=0.02 0.04 0.04; visual box size=0.02 0.04 0.04
- added link camera_link2, mass 1e-5; collision box size=0.02 0.04 0.04; visual box size=0.02 0.04 0.04
- link custom_base: geometry collision box size=0.5 0.5 1; visual box size=0.5 0.5 1
Joints:
- removed joint camera_joint
- added joint camera_joint1: type fixed, parent iiwa_link_ee, child camera_link1, origin xyz=-0.08 -0.02 0 rpy=0 -1.57 0, axis 0 1 0, mimic joint=bh_base_joint multiplier=1 offset=0
- added joint camera_joint2: type fixed, parent iiwa_link_ee, child camera_link2, origin xyz=-0.08 0.02 0 rpy=0 -1.57 0, axis 0 1 0, mimic joint=bh_base_joint multiplier=1 offset=0
- joint custom_base_iiwa_joint: origin xyz=0 0 0.822019 rpy=0 0 0 -> xyz=0 0 1 rpy=0 0 0
- joint iiwa_joint_ee: origin xyz=0 0 0.045 rpy=0 0 0 -> xyz=0 0 0 rpy=0 0 0

Commit message: move cameras further

File: src/kuka_barrett_description/urdf/hand_camera.xacro (robot description, xacro)
@@ -5,5 +5,5 @@
     <joint name="camera_joint1" type="fixed">
         <axis xyz="0 1 0" />
-        <origin xyz="-${2*camera_size} -${camera_size/2} 0" rpy="0 -1.57 0"/>
+        <origin xyz="-${3*camera_size} -${camera_size/2} 0" rpy="0 -1.57 0"/>
         <parent link="${parent}"/>
         <child link="camera_link1"/>
@@ -34,5 +34,5 @@
     <joint name="camera_joint2" type="fixed">
         <axis xyz="0 1 0" />
-        <origin xyz="-${2*camera_size} ${camera_size/2} 0" rpy="0 -1.57 0"/>
+        <origin xyz="-${3*camera_size} ${camera_size/2} 0" rpy="0 -1.57 0"/>
         <parent link="${parent}"/>
         <child link="camera_link2"/>
