Commit message: Added contact sensors to every finger of the gripper

File: src/kuka_barrett_description/urdf/kuka_barrett.xacro.urdf (robot description, URDF)
Before this commit: robot kuka_barrett, 23 links, 22 joints
Joints:
- joint camera_joint1: origin xyz=-0.08 -0.02 0 rpy=0 -1.57 0 -> xyz=-0.12 -0.02 0 rpy=0 -1.57 0
- joint camera_joint2: origin xyz=-0.08 0.02 0 rpy=0 -1.57 0 -> xyz=-0.12 0.02 0 rpy=0 -1.57 0
