Commit message: fix surgical tool collisions and path due to collisions

File: src/kuka_barrett_description/urdf/surgical_tool.xacro (robot description, xacro)
@@ -4,5 +4,5 @@
     <joint name="tool_joint" type="fixed">
         <axis xyz="0 1 0" />
-        <origin xyz="0.05 0 0.082" rpy="0 0 1.57"/>
+        <origin xyz="0.05 0 0.094" rpy="0 0 1.57"/>
         <parent link="${parent}"/>
         <child link="surgical_tool_link"/>

Commit message: draft notes of tcp-tool-tooptip frame transformations

File: src/kuka_barrett_description/urdf/surgical_tool.xacro (robot description, xacro)
@@ -35,2 +35,109 @@
   </xacro:macro>
 </robot>
+<!-- ############################################################################################################## -->
+<!-- The following are for visualization/calculation purposes only, do not uncomment if you want the robot to move! -->
+<!-- ############################################################################################################## -->
+<!-- <?xml version="1.0"?>
+<robot xmlns:xacro="http://www.ros.org/wiki/xacro">
+  <xacro:macro name="surgical_tool" params="parent">
+		<!-- 7 -> TCP -->
+		<joint name="tcp_joint" type="revolute">
+        <axis xyz="0 0 1" />
+        <origin xyz="0 0 0.094" rpy="0 0 0"/>
+        <parent link="${parent}"/>
+        <child link="tcp_link"/>
+				<limit lower="0" upper="0" effort="0" velocity="0" />
+    </joint>
+    <link name="tcp_link">
+			<collision>
+				<origin xyz="0 0 0" rpy="0 0 0"/>
+				<geometry>
+					<box size="0.06 0.06 0.03"/>
+				</geometry>
+			</collision>
+			<visual>
+				<origin xyz="0 0 0" rpy="0 0 0"/>
+				<geometry>
+					<box size="0.06 0.06 0.03"/>
+				</geometry>
+				<material name="red"/>
+			</visual>
+			<inertial>
+				<mass value="1e-5" />
+				<origin xyz="0 0 0" rpy="-1.57 0 0"/>
+				<inertia ixx="1e-6" ixy="0" ixz="0" iyy="1e-6" iyz="0" izz="1e-6" />
+			</inertial>
+			<kinematic>1</kinematic>
+    </link>
+		<gazebo reference="tcp_link">
+			<material>Gazebo/Blue</material>
+			<turnGravityOff>false</turnGravityOff>
+		</gazebo>
+		<!-- TCP -> B -->
+		<joint name="tool_joint" type="revolute">
+        <axis xyz="0 0 1" />
+        <origin xyz="0.05 0 0" rpy="1.57 0 1.57"/>
+        <parent link="tcp_link"/>
+        <child link="surgical_tool_link"/>
+				<limit lower="0" upper="0" effort="0" velocity="0" />
+    </joint>
+    <link name="surgical_tool_link">
+			<collision>
+				<origin xyz="0 0 0" rpy="-1.57 0 0"/>
+				<geometry>
+          <mesh filename="package://kuka_barrett_gazebo/objects/surgical_tool/meshes/surgical_tool_collision.stl"/>
+        </geometry>
+			</collision>
+			<visual>
+				<origin xyz="0 0 0" rpy="-1.57 0 0"/>
+				<geometry>
+          <mesh filename="package://kuka_barrett_gazebo/objects/surgical_tool/meshes/surgical_tool.stl"/>
+        </geometry>
+				<material name="red"/>
+			</visual>
+			<inertial>
+				<mass value="1e-5" />
+				<origin xyz="0 0 0" rpy="-1.57 0 0"/>
+				<inertia ixx="1e-6" ixy="0" ixz="0" iyy="1e-6" iyz="0" izz="1e-6" />
+			</inertial>
+			<kinematic>1</kinematic>
+    </link>
+		<gazebo reference="surgical_tool_link">
+			<material>Gazebo/Blue</material>
+			<turnGravityOff>false</turnGravityOff>
+		</gazebo>
+		<!-- B -> T -->
+		<joint name="tool_tip_joint" type="revolute">
+        <axis xyz="0 0 1" />
+        <origin xyz="-0.01 0.022 0.455" rpy="0 0 0"/>
+        <parent link="surgical_tool_link"/>
+        <child link="tool_tip"/>
+				<limit lower="0" upper="0" effort="0" velocity="0" />
+    </joint>
+		<link name="tool_tip">
+			<collision>
+				<origin xyz="0 0 0" rpy="0 0 0"/>
+				<geometry>
+					<box size="0.001 0.001 0.001"/>
+				</geometry>
+			</collision>
+			<visual>
+				<origin xyz="0 0 0" rpy="0 0 0"/>
+				<geometry>
+					<box size="0.001 0.001 0.001"/>
+				</geometry>
+				<material name="red"/>
+			</visual>
+			<inertial>
+				<mass value="1e-5" />
+				<origin xyz="0 0 0" rpy="-1.57 0 0"/>
+				<inertia ixx="1e-6" ixy="0" ixz="0" iyy="1e-6" iyz="0" izz="1e-6" />
+			</inertial>
+			<kinematic>1</kinematic>
+    </link>
+		<gazebo reference="tool_tip">
+			<material>Gazebo/Red</material>
+			<turnGravityOff>false</turnGravityOff>
+		</gazebo>
+  </xacro:macro>
+</robot> -->

Commit message: Caluclate transformed waypoints in planner 3a [WIP] and other minor changes

File: src/kuka_barrett_description/urdf/surgical_tool.xacro (robot description, xacro)
@@ -33,14 +33,9 @@
 			<turnGravityOff>false</turnGravityOff>
 		</gazebo>
-  </xacro:macro>
-</robot>
-<!-- ############################################################################################################## -->
-<!-- The following are for visualization/calculation purposes only, do not uncomment if you want the robot to move! -->
-<!-- ############################################################################################################## -->
-<!-- <?xml version="1.0"?>
-<robot xmlns:xacro="http://www.ros.org/wiki/xacro">
-  <xacro:macro name="surgical_tool" params="parent">
+		<!-- ############################################################################################################## -->
+		<!-- The following are for visualization/calculation purposes only, do not uncomment if you want the robot to move! -->
+		<!-- ############################################################################################################## -->
 		<!-- 7 -> TCP -->
-		<joint name="tcp_joint" type="revolute">
+		<!-- <joint name="tcp_joint" type="revolute">
         <axis xyz="0 0 1" />
         <origin xyz="0 0 0.094" rpy="0 0 0"/>
@@ -74,5 +69,4 @@
 			<turnGravityOff>false</turnGravityOff>
 		</gazebo>
-		<!-- TCP -> B -->
 		<joint name="tool_joint" type="revolute">
         <axis xyz="0 0 1" />
@@ -107,5 +101,4 @@
 			<turnGravityOff>false</turnGravityOff>
 		</gazebo>
-		<!-- B -> T -->
 		<joint name="tool_tip_joint" type="revolute">
         <axis xyz="0 0 1" />
@@ -139,5 +132,5 @@
 			<material>Gazebo/Red</material>
 			<turnGravityOff>false</turnGravityOff>
-		</gazebo>
+		</gazebo> -->
   </xacro:macro>
-</robot> -->
+</robot>
