Commit message: fix inertials and orientation

File: src/surgical_tools_description/urdf/surgical_tool.urdf (robot description, URDF)
Before this commit: robot surgical_tool, 10 links, 9 joints
Links:
- removed link grasper1_tip_L
- removed link grasper2_tip_L
- removed link tool_L
- removed link tool_base_L
- removed link tool_tip_L
- added link 0_link, mass 0.1; visual box size=0.00001 0.00001 0.00001
- link grasper1_L: mass 1e-5 -> 1
- link grasper2_L: mass 1e-5 -> 1
- link instrument_shaft_L: mass 1e-5 -> 10
- link link3_L: mass 1e-5 -> 10
- link wrist_L: mass 1e-5 -> 1
Joints:
- removed joint grasper1_tip_L
- removed joint grasper2_tip_L
- removed joint grasper_yaw_L
- removed joint tool_base_to_tool_L
- removed joint tool_base_to_tool_tip_L
- added joint insertion_L: type revolute, parent 0_link, child link3_L, origin xyz=0 0 0 rpy=1.904601 0.954344 -0.014100, axis 0 0 0, limit lower=-2 upper=2 effort=1000.0 velocity=.5
- joint grasper_joint_1_L: axis 0 0 -1 -> -0.5648    0.1427   -0.8128; origin xyz=0.012 0 0 rpy=-1.5707963267948966 0 0 -> xyz=0.00680 0.00904 -0.00452 rpy=0 0 0
- joint grasper_joint_2_L: axis 0 0 1 -> 0.5648    -0.1427   0.8128; origin xyz=0.012 0 0 rpy=-1.5707963267948966 0 0 -> xyz=0.00680 0.00904 -0.00452 rpy=0 0 0
- joint tool_roll_L: axis 0 0 -1 -> -0.6012   -0.7460    0.2864; origin xyz=0 0 0 rpy=0 0 -3.141592653589793 -> xyz=0 0 0 rpy=0 0 0
- joint wrist_joint_L: axis 0 0 -1 ->  -0.5637    0.6523    0.5067; origin xyz=0 0 0 rpy=1.5707963267948966 -1.5707963267948966 1.5707963267948966 -> xyz=0 0 0 rpy=0 0 0
